File: hw/sch_pcb/PINHOLDER01.kicad_pcb (KiCad board)
At the start: 2 copper layers, 26.9 x 50.3 mm, 5 parts, among them J1 HEADER_1x03, M3 HOLE, M4 HOLE

Commit message: uprava layoutu
Routing:
- net GND: track 40.6 -> 0.00 mm
- net /circle_0: track 6.18 -> 5.37 mm
Other:
- outline, holes or cut-outs redrawn
Changed lines of the file:
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@@
   )
   (paper "A4")
+  (title_block
+    (title "PINHOLDER01A")
+    (date "2023-04-12")
+    (rev "01A")
+    (company "www.mlab.cz")
+  )
   (layers
     (0 "F.Cu" signal)
@@
     )
   )
-  (gr_line (start 136.24 115.81) (end 136.25 65.6) (layer "Edge.Cuts") (width 0.2))
+  (gr_line (start 136.24 115.81) (end 136.24 65.51) (layer "Edge.Cuts") (width 0.2))
   (gr_line (start 109.349179 115.807146) (end 109.349179 65.515146) (layer "Edge.Cuts") (width 0.2))
   (gr_line (start 109.349179 115.807146) (end 136.24 115.81) (layer "Edge.Cuts") (width 0.2))
@@
     (effects (font (size 1.7 1.7) (thickness 0.3)))
   )
-  (segment (start 119.46 85.44) (end 119.46 89.71) (width 0.4) (layer "F.Cu") (net 1))
-  (via (at 119.46 85.44) (size 0.8) (drill 0.4) (layers "F.Cu" "B.Cu") (net 1))
-  (segment (start 119.46 85.44) (end 119.46 83.525) (width 0.4) (layer "B.Cu") (net 1))
-  (segment (start 114.175179 74.925179) (end 114.175179 70.341146) (width 0.25) (layer "B.Cu") (net 2))
-  (segment (start 114.175179 110.981146) (end 114.175179 74.925179) (width 0.25) (layer "B.Cu") (net 2))
+  (via (at 119.7 88.8) (size 0.8) (drill 0.4) (layers "F.Cu" "B.Cu") (net 1))
+  (segment (start 119.7 88.8) (end 119.46 88.56) (width 0.4) (layer "B.Cu") (net 1))
+  (segment (start 119.46 88.56) (end 119.46 83.525) (width 0.4) (layer "B.Cu") (net 1))
   (segment (start 124.48 76.52) (end 124.11 76.15) (width 0.4) (layer "F.Cu") (net 3))
   (segment (start 124.11 76.15) (end 122 76.15) (width 0.4) (layer "F.Cu") (net 3))
@@
     )
   )
-  (zone (net 0) (net_name "") (layers *.Mask) (hatch edge 0.508)
+  (zone (net 0) (net_name "") (layer "F.Mask") (hatch edge 0.508)
     (connect_pads (clearance 0.2))
     (min_thickness 0.101) (filled_areas_thickness no)
@@
     (polygon
       (pts
-        (xy 152.479179 117.331146)
-        (xy 91.569179 116.569146)
-        (xy 93.093179 59.673146)
-        (xy 152.479179 59.419146)
+        (xy 139.3 116.5)
+        (xy 105.7 116.5)
+        (xy 105.7 65)
+        (xy 139.3 65)
       )
     )
