File: hw/sch_pcb/PINHOLDER01.kicad_sch (KiCad schematic)
At the start: 5 parts, among them J1 HEADER_1x03, M3 HOLE, M4 HOLE

Commit message: uprava layoutu
Other:
- company: (none) -> www.mlab.cz
- title: (none) -> PINHOLDER01A
- moved on the sheet: TP1, TP2
Changed lines of the file:
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@@
 (kicad_sch (version 20211123) (generator eeschema)
   (paper "A4")
+  (title_block
+    (title "PINHOLDER01A")
+    (date "2023-04-12")
+    (rev "01A")
+    (company "www.mlab.cz")
+  )
   (junction (at 262.89 22.86) (diameter 0) (color 0 0 0 0)
   )
@@
     (stroke (width 0) (type solid) (color 0 0 0 0))
   )
-  (wire (pts (xy 101.6 101.6) (xy 146.05 101.6))
+  (wire (pts (xy 116.84 101.6) (xy 146.05 101.6))
     (stroke (width 0) (type default) (color 0 0 0 0))
   )
-  (polyline (pts (xy 241.3 31.75) (xy 276.86 31.75))
+  (polyline (pts (xy 254 31.75) (xy 276.86 31.75))
     (stroke (width 0) (type dash) (color 0 0 0 0))
   )
-  (polyline (pts (xy 241.3 21.59) (xy 276.86 21.59))
+  (polyline (pts (xy 254 21.59) (xy 276.86 21.59))
     (stroke (width 0) (type dash) (color 0 0 0 0))
   )
@@
     (stroke (width 0) (type solid) (color 0 0 0 0))
   )
-  (wire (pts (xy 106.68 96.52) (xy 146.05 96.52))
+  (wire (pts (xy 129.54 96.52) (xy 146.05 96.52))
     (stroke (width 0) (type default) (color 0 0 0 0))
   )
@@
     (stroke (width 0) (type dash) (color 0 0 0 0))
   )
-  (wire (pts (xy 101.6 87.63) (xy 101.6 101.6))
+  (wire (pts (xy 116.84 96.52) (xy 116.84 101.6))
     (stroke (width 0) (type default) (color 0 0 0 0))
   )
@@
     (stroke (width 0) (type solid) (color 0 0 0 0))
   )
-  (polyline (pts (xy 241.3 21.59) (xy 241.3 31.75))
+  (polyline (pts (xy 254 21.59) (xy 254 31.75))
     (stroke (width 0) (type dash) (color 0 0 0 0))
   )
-  (text "MOUNTING HOLES" (at 251.46 31.75 0)
+  (text "MOUNTING HOLES" (at 255.27 31.75 0)
     (effects (font (size 1.524 1.524)) (justify left bottom))
   )
-  (label "circle_0" (at 105.41 101.6 0)
+  (label "circle_0" (at 118.11 101.6 0)
     (effects (font (size 1.27 1.27)) (justify left bottom))
   )
-  (symbol (lib_id "Connector:TestPoint") (at 101.6 87.63 0) (unit 1)
+  (symbol (lib_id "Connector:TestPoint") (at 116.84 96.52 0) (unit 1)
     (in_bom yes) (on_board yes) (fields_autoplaced)
-    (property "Reference" "TP1" (id 0) (at 104.14 83.0579 0)
+    (property "Reference" "TP1" (id 0) (at 119.38 93.2179 0)
       (effects (font (size 1.27 1.27)) (justify left))
     )
-    (property "Value" "TestPoint" (id 1) (at 104.14 85.5979 0)
-      (effects (font (size 1.27 1.27)) (justify left))
+    (property "Value" "TestPoint" (id 1) (at 119.38 94.4879 0)
+      (effects (font (size 1.27 1.27)) (justify left) hide)
     )
-    (property "Footprint" "Mlab_CON:TestPoint_Pad_D0.5mm_noSilk" (id 2) (at 106.68 87.63 0)
+    (property "Footprint" "Mlab_CON:TestPoint_Pad_D0.5mm_noSilk" (id 2) (at 121.92 96.52 0)
       (effects (font (size 1.27 1.27)) hide)
     )
-    (property "Datasheet" "~" (id 3) (at 106.68 87.63 0)
+    (property "Datasheet" "~" (id 3) (at 121.92 96.52 0)
       (effects (font (size 1.27 1.27)) hide)
     )
-    (property "Datasheet" "~" (id 4) (at 101.6 87.63 0)
+    (property "Datasheet" "~" (id 4) (at 116.84 96.52 0)
       (effects (font (size 1.27 1.27)) hide)
     )
-    (property "Footprint" "Mlab_CON:TestPoint_Pad_D0.5mm_noSilk" (id 5) (at 101.6 87.63 0)
+    (property "Footprint" "Mlab_CON:TestPoint_Pad_D0.5mm_noSilk" (id 5) (at 116.84 96.52 0)
       (effects (font (size 1.27 1.27)) hide)
     )
-    (property "Value" "TestPoint" (id 6) (at 101.6 87.63 0)
+    (property "Value" "TestPoint" (id 6) (at 116.84 96.52 0)
       (effects (font (size 1.27 1.27)) hide)
     )
@@
   (symbol (lib_id "MLAB_HEADER:HEADER_1x03") (at 151.13 99.06 0) (unit 1)
     (in_bom yes) (on_board yes) (fields_autoplaced)
-    (property "Reference" "J1" (id 0) (at 153.67 97.79 0)
+    (property "Reference" "J1" (id 0) (at 153.67 99.695 0)
       (effects (font (size 1.524 1.524)) (justify left))
     )
     (property "Value" "HEADER_1x03" (id 1) (at 153.67 101.6 0)
-      (effects (font (size 1.524 1.524)) (justify left))
+      (effects (font (size 1.524 1.524)) (justify left) hide)
     )
     (property "Footprint" "Connector_PinHeader_2.54mm:PinHeader_1x03_P2.54mm_Vertical_SMD_Pin1Left" (id 2) (at 151.13 96.52 0)
@@
     (pin "1")
   )
-  (symbol (lib_id "Connector:TestPoint") (at 106.68 96.52 0) (unit 1)
+  (symbol (lib_id "Connector:TestPoint") (at 129.54 96.52 0) (unit 1)
     (in_bom yes) (on_board yes) (fields_autoplaced)
-    (property "Reference" "TP2" (id 0) (at 109.22 91.9479 0)
+    (property "Reference" "TP2" (id 0) (at 132.08 93.2179 0)
       (effects (font (size 1.27 1.27)) (justify left))
     )
-    (property "Value" "TestPoint" (id 1) (at 109.22 94.4879 0)
-      (effects (font (size 1.27 1.27)) (justify left))
+    (property "Value" "TestPoint" (id 1) (at 132.08 94.4879 0)
+      (effects (font (size 1.27 1.27)) (justify left) hide)
     )
-    (property "Footprint" "TestPoint:TestPoint_Keystone_5019_Minature" (id 2) (at 111.76 96.52 0)
+    (property "Footprint" "TestPoint:TestPoint_Keystone_5019_Minature" (id 2) (at 134.62 96.52 0)
       (effects (font (size 1.27 1.27)) hide)
     )
-    (property "Datasheet" "~" (id 3) (at 111.76 96.52 0)
+    (property "Datasheet" "~" (id 3) (at 134.62 96.52 0)
       (effects (font (size 1.27 1.27)) hide)
     )
-    (property "Datasheet" "~" (id 4) (at 106.68 96.52 0)
+    (property "Datasheet" "~" (id 4) (at 129.54 96.52 0)
       (effects (font (size 1.27 1.27)) hide)
     )
-    (property "Footprint" "Mlab_CON:TestPoint_Pad_D0.5mm_noSilk" (id 5) (at 106.68 96.52 0)
+    (property "Footprint" "Mlab_CON:TestPoint_Pad_D0.5mm_noSilk" (id 5) (at 129.54 96.52 0)
       (effects (font (size 1.27 1.27)) hide)
     )
-    (property "Value" "TestPoint" (id 6) (at 106.68 96.52 0)
+    (property "Value" "TestPoint" (id 6) (at 129.54 96.52 0)
       (effects (font (size 1.27 1.27)) hide)
     )
