File: hw/sch_pcb/PINHOLDER03.kicad_pcb (KiCad board)
At the start: 2 copper layers, 50.3 x 30 mm, 9 parts, among them J1 HEADER_1x03, J2 HEADER_1x02, M1 HOLE, M2 HOLE, M3 HOLE, M4 HOLE

Commit message: Edit PCB
Other:
- rule pad_to_mask_clearance: 0 -> 0.2
Changed lines of the file:
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@@
   )
   (setup
-    (pad_to_mask_clearance 0)
+    (stackup
+      (layer "F.SilkS" (type "Top Silk Screen"))
+      (layer "F.Paste" (type "Top Solder Paste"))
+      (layer "F.Mask" (type "Top Solder Mask") (thickness 0.01))
+      (layer "F.Cu" (type "copper") (thickness 0.035))
+      (layer "dielectric 1" (type "core") (thickness 1.51) (material "FR4") (epsilon_r 4.5) (loss_tangent 0.02))
+      (layer "B.Cu" (type "copper") (thickness 0.035))
+      (layer "B.Mask" (type "Bottom Solder Mask") (thickness 0.01))
+      (layer "B.Paste" (type "Bottom Solder Paste"))
+      (layer "B.SilkS" (type "Bottom Silk Screen"))
+      (copper_finish "None")
+      (dielectric_constraints no)
+    )
+    (pad_to_mask_clearance 0.2)
     (aux_axis_origin 149.61 76.48)
     (pcbplotparams
@@
     (pts (xy 195.076 101.626) (xy 195.076 71.654))
     (height 4.314)
-    (gr_text "29,9720 mm" (at 198.24 86.64 90) (layer "Cmts.User")
+    (gr_text "29.9720 mm" (at 198.24 86.64 90) (layer "Cmts.User")
       (effects (font (size 1 1) (thickness 0.15)))
     )
@@
     (pts (xy 144.784 101.626) (xy 195.076 101.626))
     (height 3.784)
-    (gr_text "50,2920 mm" (at 169.93 104.26) (layer "Cmts.User")
-      (effects (font (size 1 1) (thickness 0.15)))
-    )
+    (gr_text "50.2920 mm" (at 169.93 104.26) (layer "Cmts.User")
+      (effects (font (size 1 1) (thickness 0.15)))
+    )
